File: PCB/OBC/coms.kicad_sch (KiCad schematic)
At the start: 25 parts, among them U4 STM32F405RGTx

Commit message: bomkicad
Parts:
- R10, R9: LCSC Part Name (none) -> C19701189
- R8: LCSC Part Name (none) -> C19679468
- XTAL2: LCSC Part Name (none) -> C6942002
Changed lines of the file:
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@@
 			)
 		)
+		(property "LCSC Part Name" "C19701189"
+			(at 140.97 171.45 0)
+			(effects
+				(font
+					(size 1.27 1.27)
+				)
+			)
+		)
 		(pin "2"
 		)
@@
 			)
 		)
+		(property "LCSC Part Name" "C19701189"
+			(at 129.54 171.45 0)
+			(effects
+				(font
+					(size 1.27 1.27)
+				)
+			)
+		)
 		(pin "2"
 		)
@@
 			)
 		)
+		(property "LCSC Part Name" "C6942002"
+			(at 31.75 66.04 0)
+			(effects
+				(font
+					(size 1.27 1.27)
+				)
+			)
+		)
 		(pin "1"
 		)
@@
 			)
 		)
+		(property "LCSC Part Name" "C19679468"
+			(at 43.18 177.8 0)
+			(effects
+				(font
+					(size 1.27 1.27)
+				)
+			)
+		)

Commit message: Revert "Merge branch 'main' of https://github.com/HernanIbarra60/OBC-"
This reverts commit 45b73800fdf824c252c0947f7787583bb3814567, reversing
changes made to df5dc6ac9bf84d542dd85559211e3d40553a5f31.
Parts:
- added COMS1: Conn_01x05, Connector_PinHeader_2.54mm:PinHeader_1x05_P2.54mm_Vertical_SMD_Pin1Right, symbol Connector_Generic:Conn_01x05
- C20, C24, C27, C30, C31: LCSC Part Name C1591 -> C15725
- FB2: Mouser (none) -> 81-BLM21HE601SN1L
- R10, R9: LCSC Part Name C19701189 -> C2930157; now in the parts list
- R8: LCSC Part Name C19679468 -> C2907219; now in the parts list
- SwBoot2: LCSC Part Name C5962834 -> C22401620
- XTAL2: LCSC Part Name C6942002 -> (none); Mouser (none) -> 520-8012-30BQ-JES-TR
Connections:
- net +3V3: now also COMS1.1 (Pin_1)
- net GND: now also COMS1.5 (Pin_5)
- net MainComs_RX: now reaches U4.14 (PA0)
- net MainComs_TX: now reaches U4.15 (PA1)
- net ObcComs_TX: now reaches U4.51 (PC10)
- net ComsOBC_RX: now reaches U4.52 (PC11)
- net ComMem_SCK: now reaches U4.55 (PB3)
- net ComMem_MISO: now reaches U4.56 (PB4)
- net ComMem_MOSI: now reaches U4.57 (PB5)
- net Coms_RX: no longer names the net of U4.42 (PA9)
- net Coms_TX: no longer names the net of U4.43 (PA10)
- net SWCLK2 renamed SWCLK_Com
- net SWCLK_Com: now also COMS1.2 (Pin_2)
- net SWDIO2 renamed SWDIO_Com
- net SWDIO_Com: now also COMS1.3 (Pin_3)
- net SWD_NRST renamed ComsRESET
- net ComsRESET: now also COMS1.4 (Pin_4)
Other:
- moved on the sheet: D4, D5, R10, R9
