File: PCB/OBC/main.kicad_sch (KiCad schematic)
At the start: 36 parts, among them J3 USB_C_Receptacle_USB2.0_16P, U1 STM32F405RGTx, U2 SN65HVD230DR, U3 USBLC6-2SC6

Commit message: bomkicad
Parts:
- J3: LCSC Part Name (none) -> C2765186
- R1, R6: LCSC Part Name (none) -> C19679468
- R2, R3: LCSC Part Name (none) -> C19701189
- R7: LCSC Part Name (none) -> C19706317
- XTAL1: LCSC Part Name (none) -> C6942002
Changed lines of the file:
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@@
 			)
 		)
+		(property "LCSC Part Name" "C19679468"
+			(at 43.18 176.53 0)
+			(effects
+				(font
+					(size 1.27 1.27)
+				)
+			)
+		)
 		(pin "1"
 		)
@@
 			)
 		)
+		(property "LCSC Part Name" "C19706317"
+			(at 255.27 135.89 0)
+			(effects
+				(font
+					(size 1.27 1.27)
+				)
+			)
+		)
 		(pin "1"
 		)
@@
 			)
 		)
+		(property "LCSC Part Name" "C19679468"
+			(at 245.11 125.73 0)
+			(effects
+				(font
+					(size 1.27 1.27)
+				)
+			)
+		)
 		(pin "1"
 		)
@@
 			)
 		)
+		(property "LCSC Part Name" "C2765186"
+			(at 198.12 39.37 0)
+			(effects
+				(font
+					(size 1.27 1.27)
+				)
+			)
+		)
 		(pin "B6"
 		)
@@
 			)
 		)
+		(property "LCSC Part Name" "C6942002"
+			(at 40.64 78.74 0)
+			(effects
+				(font
+					(size 1.27 1.27)
+				)
+			)
+		)
 		(pin "1"
 		)
@@
 			)
 		)
+		(property "LCSC Part Name" "C19701189"
+			(at 140.97 170.18 0)
+			(effects
+				(font
+					(size 1.27 1.27)
+				)
+			)
+		)
 		(pin "2"
 		)
@@
 			)
 		)
+		(property "LCSC Part Name" "C19701189"
+			(at 129.54 170.18 0)
+			(effects
+				(font
+					(size 1.27 1.27)
+				)
+			)
+		)

Commit message: Revert "Merge branch 'main' of https://github.com/HernanIbarra60/OBC-"
This reverts commit 45b73800fdf824c252c0947f7787583bb3814567, reversing
changes made to df5dc6ac9bf84d542dd85559211e3d40553a5f31.
Parts:
- added MAIN1: Conn_01x05, Connector_PinHeader_2.54mm:PinHeader_1x05_P2.54mm_Vertical_SMD_Pin1Right, symbol Connector_Generic:Conn_01x05
- added R15, R21: 4.7k, Resistor_SMD:R_0805_2012Metric_Pad1.20x1.40mm_HandSolder, symbol Device:R
- C13, C14, C16, C4, C9: LCSC Part Name C1591 -> C15725
- FB1: Mouser (none) -> 81-BLM21HE601SN1L
- J3: LCSC Part Name C2765186 -> (none); Mouser (none) -> 640-USB4940-00-A
- R1: LCSC Part Name C19679468 -> C2907219; now in the parts list
- R2, R3: LCSC Part Name C19701189 -> C2930157; now in the parts list
- R6: footprint (none) -> Resistor_SMD:R_0805_2012Metric_Pad1.20x1.40mm_HandSolder; LCSC Part Name C19679468 -> C2907219
- R7: footprint (none) -> Resistor_SMD:R_0805_2012Metric_Pad1.20x1.40mm_HandSolder; LCSC Part Name C19706317 -> C17437
- SwBoot1: LCSC Part Name C5962834 -> C22401620
- U3: LCSC Part Name C2969755 -> C7519
- XTAL1: LCSC Part Name C6942002 -> (none); Mouser (none) -> 520-8012-30BQ-JES-TR
Connections:
- net +3V3: now also MAIN1.1 (Pin_1), R15.1, R21.1
- net Can_RX: now also U1.61 (PB8)
- net Can_TX: now also U1.62 (PB9)
- net GND: now also MAIN1.5 (Pin_5)
- net EnMuxPy: now reaches U1.51 (PC10)
- net EnMemPy: now reaches U1.52 (PC11)
- net PY2_SCK: now reaches U1.55 (PB3)
- net PY2_MISO: now reaches U1.56 (PB4)
- net PY2_MOSI: now reaches U1.57 (PB5)
- net I2C_SCL: now reaches U1.58 (PB6)
- net I2C_SCL: now also R15.2
- net I2C_SDA: now reaches U1.59 (PB7)
- net I2C_SDA: now also R21.2
- net BOOT0 renamed BootMain
- net Coms_RX renamed MainComs_RX
- net Coms_TX renamed MainComs_TX
- net Rst_RX renamed MainPwr_RX
- net Rst_TX renamed MainPwr_TX
- net SWCLK1 renamed SWCLK
- net SWCLK: now also MAIN1.2 (Pin_2)
- net SWDIO1 renamed SWDIO
- net SWDIO: now also MAIN1.3 (Pin_3)
- net SWD_NRST renamed SWNRST
- net SWNRST: now also MAIN1.4 (Pin_4)
- no-connect marks 10 -> 8
Other:
- note added: "SWD"
- moved on the sheet: R6, R7, U2
