File: PCB/OBC/memory.kicad_sch (KiCad schematic)
At the start: 14 parts, among them U10 TMUX1574PWR, U11 W25Q128JVSIQ, U12 TMUX1574PWR, U9 W25Q128JVSIQ

Commit message: bomkicad
Parts:
- C53, C54, C56, C58: LCSC Part Name (none) -> C49678
- C55, C57: LCSC Part Name (none) -> C28323
- R16, R17, R18, R19: LCSC Part Name (none) -> C19679468
Changed lines of the file:
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@@
+			)
+		)
+		(property "LCSC Part Name" "C19679468"
+			(at 254 80.01 0)
+			(effects
+				(font
+					(size 1.27 1.27)
+				)
 			)
 		)
@@
 			)
 		)
+		(property "LCSC Part Name" "C28323"
+			(at 212.09 62.23 0)
+			(effects
+				(font
+					(size 1.27 1.27)
+				)
+			)
+		)
 		(pin "1"
 		)
@@
 				)
 				(hide yes)
+			)
+		)
+		(property "LCSC Part Name" "C28323"
+			(at 142.24 72.39 0)
+			(effects
+				(font
+					(size 1.27 1.27)
+				)
 			)
 		)
@@
 				)
 				(hide yes)
+			)
+		)
+		(property "LCSC Part Name" "C49678"
+			(at 129.54 72.39 0)
+			(effects
+				(font
+					(size 1.27 1.27)
+				)
 			)
 		)
@@
 			)
 		)
+		(property "LCSC Part Name" "C49678"
+			(at 269.24 127 0)
+			(effects
+				(font
+					(size 1.27 1.27)
+				)
+			)
+		)
 		(pin "2"
 		)
@@
 			)
 		)
+		(property "LCSC Part Name" "C49678"
+			(at 199.39 62.23 0)
+			(effects
+				(font
+					(size 1.27 1.27)
+				)
+			)
+		)
 		(pin "1"
 		)
@@
 			)
 		)
+		(property "LCSC Part Name" "C19679468"
+			(at 34.29 74.93 0)
+			(effects
+				(font
+					(size 1.27 1.27)
+				)
+			)
+		)
 		(pin "2"
 		)
@@
 			)
 		)
+		(property "LCSC Part Name" "C19679468"
+			(at 109.22 67.31 0)
+			(effects
+				(font
+					(size 1.27 1.27)
+				)
+			)
+		)
 		(pin "1"
 		)
@@
 			)
 		)
+		(property "LCSC Part Name" "C49678"
+			(at 119.38 116.84 0)
+			(effects
+				(font
+					(size 1.27 1.27)
+				)
+			)
+		)
 		(pin "2"
 		)
@@
 			)
 		)
+		(property "LCSC Part Name" "C19679468"
+			(at 173.99 88.9 0)
+			(effects
+				(font
+					(size 1.27 1.27)
+				)
+			)
+		)

Commit message: Revert "Merge branch 'main' of https://github.com/HernanIbarra60/OBC-"
This reverts commit 45b73800fdf824c252c0947f7787583bb3814567, reversing
changes made to df5dc6ac9bf84d542dd85559211e3d40553a5f31.
Parts:
- removed U12: TMUX1574PWR, TMUX1574PWR:PWP16_2P31X2P46_TEX, symbol TMUX1574PWR:TMUX1574PWR
- added U8: TMUX1574PWR, TMUX1574PWR:SOP65P640X120-16N, symbol TMUX1574PWR:TMUX1574PWR
- C53, C54, C56, C58: LCSC Part Name C49678 -> C1711
- C55: footprint XTAL_NX3215SA_NDK:XTAL_NX3215SA_NDK -> Capacitor_SMD:C_0805_2012Metric_Pad1.18x1.45mm_HandSolder
- C57: footprint TMUX1574PWR:PWP16_2P31X2P46_TEX -> Capacitor_SMD:C_0805_2012Metric_Pad1.18x1.45mm_HandSolder
- R16, R17, R18, R19: footprint (none) -> Resistor_SMD:R_0805_2012Metric_Pad1.20x1.40mm_HandSolder; LCSC Part Name C19679468 -> C2907219
- U10: footprint TMUX1574PWR:PWP16_2P31X2P46_TEX -> TMUX1574PWR:SOP65P640X120-16N
Connections:
- net select_py is gone; now on net select_coms: U10.1 (SEL)
- net +3V3: now also U8.16 (VDD)
- net GND: now also U8.15 (~{EN}), U8.8 (GND); no longer U9.1 (/CS)
- net coms_flash_clk_m: now also U10.9 (D3)
- net coms_flash_miso_m: now also U10.4 (D1)
- net coms_flash_mosi_m: now also U10.7 (D2)
- net py_flash_clk_m: now also U8.9 (D3); no longer U10.12 (D4)
- net py_flash_miso_m: now also U8.4 (D1); no longer U10.7 (D2)
- net py_flash_mosi_m: now also U8.7 (D2); no longer U10.9 (D3)
- net SPI_SCK: now reaches U10.10 (S3B)
- net ComMem_SCK: now reaches U10.11 (S3A)
- net ComMem_MISO: now reaches U10.2 (S1A)
- net SPI_MISO: now reaches U10.3 (S1B)
- net ComMem_MOSI: now reaches U10.5 (S2A)
- net SPI_MOSI: now reaches U10.6 (S2B)
- new net EnMemPy: U9.1 (/CS)
- new net EnMuxPy: U8.1 (SEL)
- new net PY2_MISO: U8.2 (S1A)
- new net PY2_MOSI: U8.5 (S2A)
- new net PY2_SCK: U8.11 (S3A)
- no-connect marks 2 -> 9
Other:
- moved on the sheet: C53
