File: PCB/OBC/memory.kicad_sch (KiCad schematic)
At the start: 14 parts, among them U10 TMUX1574PWR, U11 W25Q128JVSIQ, U8 TMUX1574PWR, U9 W25Q128JVSIQ

Commit message: Coms memory finished
Connections:
- net cs_mem_py: no longer U10.12 (D4), U11.1 (/CS)
- new net cs_mem_coms: U10.12 (D4), U11.1 (/CS)
Changed lines of the file:
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@@
 		)
 	)
-	(label "cs_mem_py"
+	(label "cs_mem_coms"
 		(at 228.6 118.11 0)
 		(effects
@@
 		)
 	)
-	(label "cs_mem_py"
+	(label "cs_mem_coms"
 		(at 176.53 71.12 180)
 		(effects
