File: PCB/OBC/OBC.kicad_pcb (KiCad board)
At the start: 2 copper layers, 1 part

Commit message: New
Parts:
- added C1: 4.7u, Capacitor_SMD:C_0805_2012Metric_Pad1.18x1.45mm_HandSolder, F.Cu at (31.5, 70.9)
- added C10: 15pF, Capacitor_SMD:C_0603_1608Metric_Pad1.08x0.95mm_HandSolder, F.Cu at (36.1, 83.2)
- added C11: 100nF, Capacitor_SMD:C_0805_2012Metric_Pad1.18x1.45mm_HandSolder, F.Cu at (31.5, 83.0)
- added C12: 2.2uF, Capacitor_SMD:C_0805_2012Metric_Pad1.18x1.45mm_HandSolder, F.Cu at (31.5, 86.0)
- added C13: 100nF, Capacitor_SMD:C_0603_1608Metric_Pad1.08x0.95mm_HandSolder, F.Cu at (36.1, 85.7)
- added C14: 100nF, Capacitor_SMD:C_0603_1608Metric_Pad1.08x0.95mm_HandSolder, F.Cu at (36.1, 88.2)
- added C15: 2.2uF, Capacitor_SMD:C_0805_2012Metric_Pad1.18x1.45mm_HandSolder, F.Cu at (31.5, 89.0)
- added C16: 100nF, Capacitor_SMD:C_0603_1608Metric_Pad1.08x0.95mm_HandSolder, F.Cu at (36.1, 90.7)
- added C17: 1uF, Capacitor_SMD:C_0805_2012Metric_Pad1.18x1.45mm_HandSolder, F.Cu at (31.5, 92.0)
- added C18: 4.7u, Capacitor_SMD:C_0805_2012Metric_Pad1.18x1.45mm_HandSolder, F.Cu at (31.5, 104.5)
- added C19: 15pF, Capacitor_SMD:C_0603_1608Metric_Pad1.08x0.95mm_HandSolder, F.Cu at (36.1, 104.2)
- added C2: 15pF, Capacitor_SMD:C_0603_1608Metric_Pad1.08x0.95mm_HandSolder, F.Cu at (36.1, 70.7)
- added C20: 100nF, Capacitor_SMD:C_0603_1608Metric_Pad1.08x0.95mm_HandSolder, F.Cu at (36.1, 106.7)
- added C21: 10uF, Capacitor_SMD:C_0805_2012Metric_Pad1.18x1.45mm_HandSolder, F.Cu at (31.5, 107.5)
- added C22: 100nF, Capacitor_SMD:C_0805_2012Metric_Pad1.18x1.45mm_HandSolder, F.Cu at (31.5, 110.5)
- added C23: 100nF, Capacitor_SMD:C_0805_2012Metric_Pad1.18x1.45mm_HandSolder, F.Cu at (31.5, 113.5)
- added C24: 100nF, Capacitor_SMD:C_0603_1608Metric_Pad1.08x0.95mm_HandSolder, F.Cu at (36.1, 109.2)
- added C25: 15pF, Capacitor_SMD:C_0603_1608Metric_Pad1.08x0.95mm_HandSolder, F.Cu at (36.1, 111.8)
- added C26: 100nF, Capacitor_SMD:C_0805_2012Metric_Pad1.18x1.45mm_HandSolder, F.Cu at (31.5, 116.5)
- added C27: 100nF, Capacitor_SMD:C_0603_1608Metric_Pad1.08x0.95mm_HandSolder, F.Cu at (36.1, 114.3)
- added C28: 2.2uF, Capacitor_SMD:C_0805_2012Metric_Pad1.18x1.45mm_HandSolder, F.Cu at (31.5, 119.5)
- added C29: 2.2uF, Capacitor_SMD:C_0805_2012Metric_Pad1.18x1.45mm_HandSolder, F.Cu at (31.5, 122.5)
- added C3: 12pF, Capacitor_SMD:C_0603_1608Metric_Pad1.08x0.95mm_HandSolder, F.Cu at (36.1, 73.2)
- added C30: 100nF, Capacitor_SMD:C_0603_1608Metric_Pad1.08x0.95mm_HandSolder, F.Cu at (36.1, 116.8)
- added C31: 100nF, Capacitor_SMD:C_0603_1608Metric_Pad1.08x0.95mm_HandSolder, F.Cu at (36.1, 119.3)
- added C32: 1uF, Capacitor_SMD:C_0805_2012Metric_Pad1.18x1.45mm_HandSolder, F.Cu at (31.5, 125.5)
- added C33: 15pF, Capacitor_SMD:C_0603_1608Metric_Pad1.08x0.95mm_HandSolder, F.Cu at (66.9, 70.7)
- added C34: 4.7u, Capacitor_SMD:C_0805_2012Metric_Pad1.18x1.45mm_HandSolder, F.Cu at (62.3, 70.9)
- added C35: 100nF, Capacitor_SMD:C_0603_1608Metric_Pad1.08x0.95mm_HandSolder, F.Cu at (66.9, 73.2)
- added C36: 10uF, Capacitor_SMD:C_0805_2012Metric_Pad1.18x1.45mm_HandSolder, F.Cu at (62.3, 73.9)
- added C37: 100nF, Capacitor_SMD:C_0805_2012Metric_Pad1.18x1.45mm_HandSolder, F.Cu at (62.3, 76.9)
- added C38: 100nF, Capacitor_SMD:C_0805_2012Metric_Pad1.18x1.45mm_HandSolder, F.Cu at (62.3, 79.9)
- added C39: 15pF, Capacitor_SMD:C_0603_1608Metric_Pad1.08x0.95mm_HandSolder, F.Cu at (66.9, 75.7)
- added C4: 100nF, Capacitor_SMD:C_0603_1608Metric_Pad1.08x0.95mm_HandSolder, F.Cu at (36.1, 75.7)
- added C40: 100nF, Capacitor_SMD:C_0603_1608Metric_Pad1.08x0.95mm_HandSolder, F.Cu at (66.9, 78.2)
- added C41: 100nF, Capacitor_SMD:C_0805_2012Metric_Pad1.18x1.45mm_HandSolder, F.Cu at (62.3, 83.0)
- added C42: 2.2uF, Capacitor_SMD:C_0805_2012Metric_Pad1.18x1.45mm_HandSolder, F.Cu at (62.3, 86.0)
- added C43: 100nF, Capacitor_SMD:C_0603_1608Metric_Pad1.08x0.95mm_HandSolder, F.Cu at (66.9, 80.7)
- added C44: 2.2uF, Capacitor_SMD:C_0805_2012Metric_Pad1.18x1.45mm_HandSolder, F.Cu at (62.3, 89.0)
- added C45: 100nF, Capacitor_SMD:C_0603_1608Metric_Pad1.08x0.95mm_HandSolder, F.Cu at (66.9, 83.2)
- added C46: 100nF, Capacitor_SMD:C_0603_1608Metric_Pad1.08x0.95mm_HandSolder, F.Cu at (66.9, 85.7)
- added C47: 1uF, Capacitor_SMD:C_0805_2012Metric_Pad1.18x1.45mm_HandSolder, F.Cu at (62.3, 92.0)
- added C5: 10uF, Capacitor_SMD:C_0805_2012Metric_Pad1.18x1.45mm_HandSolder, F.Cu at (31.5, 73.9)
- added C51: 100nF, Capacitor_SMD:C_0805_2012Metric_Pad1.18x1.45mm_HandSolder, F.Cu at (80.3, 122.7)
- added C52: 100nF, Capacitor_SMD:C_0805_2012Metric_Pad1.18x1.45mm_HandSolder, F.Cu at (80.3, 125.7)
- added C53: 100nF, Capacitor_SMD:C_0805_2012Metric_Pad1.18x1.45mm_HandSolder, F.Cu at (81.9, 100.4)
- added C54: 100nF, Capacitor_SMD:C_0805_2012Metric_Pad1.18x1.45mm_HandSolder, F.Cu at (81.9, 103.4)
- added C55: 1uF, XTAL_NX3215SA_NDK:XTAL_NX3215SA_NDK, F.Cu at (72.5, 114.5)
- added C56: 100nF, Capacitor_SMD:C_0805_2012Metric_Pad1.18x1.45mm_HandSolder, F.Cu at (81.9, 106.4)
- added C57: 1uF, TMUX1574PWR:PWP16_2P31X2P46_TEX, F.Cu at (64.4, 102.3)
- added C58: 100nF, Capacitor_SMD:C_0805_2012Metric_Pad1.18x1.45mm_HandSolder, F.Cu at (81.9, 109.4)
- added C59: 10uF, Capacitor_SMD:C_0805_2012Metric_Pad1.18x1.45mm_HandSolder, F.Cu at (80.3, 128.7)
- added C6: 100nF, Capacitor_SMD:C_0805_2012Metric_Pad1.18x1.45mm_HandSolder, F.Cu at (31.5, 76.9)
- added C60: 150uF, Capacitor_SMD:C_Elec_6.3x7.7, F.Cu at (64.8, 134.4)
- added C7: 12pF, Capacitor_SMD:C_0603_1608Metric_Pad1.08x0.95mm_HandSolder, F.Cu at (36.1, 78.2)
- added C8: 100nF, Capacitor_SMD:C_0805_2012Metric_Pad1.18x1.45mm_HandSolder, F.Cu at (31.5, 79.9)
- added C9: 100nF, Capacitor_SMD:C_0603_1608Metric_Pad1.08x0.95mm_HandSolder, F.Cu at (36.1, 80.7)
- added D1: LED, LED_SMD:LED_0805_2012Metric_Pad1.15x1.40mm_HandSolder, F.Cu at (54.7, 85.7)
- added D2: LED, LED_SMD:LED_0805_2012Metric_Pad1.15x1.40mm_HandSolder, F.Cu at (54.7, 88.7)
- added D3: D_Schottky, Diode_SMD:D_SOD-323_HandSoldering, F.Cu at (40.8, 99.5)
- added D4: LED, LED_SMD:LED_0805_2012Metric_Pad1.15x1.40mm_HandSolder, F.Cu at (53.0, 125.9)
- added D5: LED, LED_SMD:LED_0805_2012Metric_Pad1.15x1.40mm_HandSolder, F.Cu at (53.0, 128.9)
- added D6: LED, LED_SMD:LED_0805_2012Metric_Pad1.15x1.40mm_HandSolder, F.Cu at (83.8, 92.3)
- added D7: LED, LED_SMD:LED_0805_2012Metric_Pad1.15x1.40mm_HandSolder, F.Cu at (83.8, 95.4)
- added FB1: FerriteBead, Capacitor_SMD:C_0805_2012Metric_Pad1.18x1.45mm_HandSolder, F.Cu at (31.5, 95.0)
- added FB2: FerriteBead, Capacitor_SMD:C_0805_2012Metric_Pad1.18x1.45mm_HandSolder, F.Cu at (31.5, 128.6)
- added FB3: FerriteBead, Capacitor_SMD:C_0805_2012Metric_Pad1.18x1.45mm_HandSolder, F.Cu at (62.3, 95.0)
- added IC1: TPS2553QDBVRQ1, OCP_TPS2553QDBVRQ1:SOT95P280X145-6N, F.Cu at (80.4, 137.3)
- added J2: Conn_01x04, Connector_PinSocket_2.54mm:PinSocket_1x04_P2.54mm_Vertical_SMD_Pin1Left, F.Cu at (61.2, 54.3)
- added J4: SWD, Connector_PinHeader_2.54mm:PinHeader_1x05_P2.54mm_Vertical_SMD_Pin1Left, F.Cu at (73.8, 137.8)
- added LSE1: Crystal, XTAL_NX3215SA_NDK:XTAL_NX3215SA_NDK, F.Cu at (50.2, 97.2)
- added R1: 10k, Resistor_SMD:R_0805_2012Metric_Pad1.20x1.40mm_HandSolder, F.Cu at (40.6, 70.9)
- added R10: 330, Resistor_SMD:R_0805_2012Metric_Pad1.20x1.40mm_HandSolder, F.Cu at (40.6, 124.8)
- added R11: 10k, Resistor_SMD:R_0805_2012Metric_Pad1.20x1.40mm_HandSolder, F.Cu at (71.4, 85.3)
- added R12: 330, Resistor_SMD:R_0805_2012Metric_Pad1.20x1.40mm_HandSolder, F.Cu at (71.4, 88.3)
- added R13: 330, Resistor_SMD:R_0805_2012Metric_Pad1.20x1.40mm_HandSolder, F.Cu at (71.4, 91.2)
- added R2: 330, Resistor_SMD:R_0805_2012Metric_Pad1.20x1.40mm_HandSolder, F.Cu at (40.6, 73.8)
- added R20: 10K, Resistor_SMD:R_0805_2012Metric_Pad1.20x1.40mm_HandSolder, F.Cu at (80.2, 141.1)
- added R21: 26.1K, Resistor_SMD:R_0805_2012Metric_Pad1.20x1.40mm_HandSolder, F.Cu at (80.2, 144.1)
- added R3: 330, Resistor_SMD:R_0805_2012Metric_Pad1.20x1.40mm_HandSolder, F.Cu at (40.6, 76.8)
- added R4: 5k1, Resistor_SMD:R_0805_2012Metric_Pad1.20x1.40mm_HandSolder, F.Cu at (40.6, 79.7)
- added R5: 5k1, Resistor_SMD:R_0805_2012Metric_Pad1.20x1.40mm_HandSolder, F.Cu at (40.6, 82.7)
- added R8: 10k, Resistor_SMD:R_0805_2012Metric_Pad1.20x1.40mm_HandSolder, F.Cu at (40.6, 118.9)
- added R9: 330, Resistor_SMD:R_0805_2012Metric_Pad1.20x1.40mm_HandSolder, F.Cu at (40.6, 121.8)
- added SW1: SS-23D03-G080, SlideSwitch2P3T:SW-TH_SS-23D03-G080, F.Cu at (116.1, 111.1)
- added SwBoot1: SW_Nidec_CAS-120A1, Button_Switch_SMD:Nidec_Copal_CAS-120A, F.Cu at (49.5, 87.6)
- added SwBoot2: SW_Nidec_CAS-120A1, Button_Switch_SMD:Nidec_Copal_CAS-120A, F.Cu at (53.3, 120.9)
- added SwBoot3: SW_Nidec_CAS-120A1, Button_Switch_SMD:Nidec_Copal_CAS-120A, F.Cu at (84.1, 87.3)
- added SwReset1: SW_Push, Button_Switch_SMD:SW_Push_SPST_NO_Alps_SKRK, F.Cu at (50.1, 93.3)
- added SwReset2: SW_Push, Button_Switch_SMD:SW_Push_SPST_NO_Alps_SKRK, F.Cu at (46.3, 126.9)
- added SwReset3: SW_Push, Button_Switch_SMD:SW_Push_SPST_NO_Alps_SKRK, F.Cu at (77.1, 93.3)
- added U1: STM32F405RGTx, Package_QFP:LQFP-64_10x10mm_P0.5mm, F.Cu at (50.2, 76.6)
- added U10: TMUX1574PWR, TMUX1574PWR:PWP16_2P31X2P46_TEX, F.Cu at (64.4, 109.0)
- added U11: W25Q128JVSIQ, W25Q128JVS:SOIC_128JVSIQ_WIN, F.Cu at (74.2, 109.4)
- added U12: TMUX1574PWR, TMUX1574PWR:PWP16_2P31X2P46_TEX, F.Cu at (64.4, 115.8)
- added U2: SN65HVD230DR, SN65HVD230DR:D8, F.Cu at (42.5, 87.5)
- added U3: USBLC6-2SC6, Package_TO_SOT_SMD:SOT-23-6, F.Cu at (55.3, 98.0)
- added U4: STM32F405RGTx, Package_QFP:LQFP-64_10x10mm_P0.5mm, F.Cu at (45.5, 110.2)
- added U5: STM32F405RGTx, Package_QFP:LQFP-64_10x10mm_P0.5mm, F.Cu at (76.3, 76.6)
- added U6: MAX6369KA+T, MAX6369KA+T:21-0078H_MXM, F.Cu at (80.5, 132.7)
- added U8: AMS1117-3.3, Package_TO_SOT_SMD:SOT-223-3_TabPin2, F.Cu at (64.8, 142.7)
- added U9: W25Q128JVSIQ, W25Q128JVS:SOIC_128JVSIQ_WIN, F.Cu at (74.2, 102.4)
- added XTAL1: ECS-80-12-30BQ-JES-TR, ECS-80-12-30BQ-JES-TR:ECS-80-12_ECS, F.Cu at (43.2, 94.5)
- added XTAL2: ECS-80-12-30BQ-JES-TR, ECS-80-12-30BQ-JES-TR:ECS-80-12_ECS, F.Cu at (48.0, 121.2)
- added XTAL3: ECS-80-12-30BQ-JES-TR, ECS-80-12-30BQ-JES-TR:ECS-80-12_ECS, F.Cu at (78.8, 87.6)
Routing:
- net (no net): track 34.5 -> 1.75 mm

Commit message: BOM terminado
Parts:
- removed C52: 100nF, Capacitor_SMD:C_0805_2012Metric_Pad1.18x1.45mm_HandSolder
- removed C59: 10uF, Capacitor_SMD:C_0805_2012Metric_Pad1.18x1.45mm_HandSolder
- removed J2: Conn_01x04, Connector_PinSocket_2.54mm:PinSocket_1x04_P2.54mm_Vertical_SMD_Pin1Left
- removed J4: SWD, Connector_PinHeader_2.54mm:PinHeader_1x05_P2.54mm_Vertical_SMD_Pin1Left
- removed R21: 26.1K, Resistor_SMD:R_0805_2012Metric_Pad1.20x1.40mm_HandSolder
- removed REF**: PinHeader_2x24_P2.54mm_Vertical, Connector_PinHeader_2.54mm:PinHeader_2x24_P2.54mm_Vertical
- removed SW1: SS-23D03-G080, SlideSwitch2P3T:SW-TH_SS-23D03-G080
- removed U8: AMS1117-3.3, Package_TO_SOT_SMD:SOT-223-3_TabPin2
- added C48: 100nF, Capacitor_SMD:C_0805_2012Metric_Pad1.18x1.45mm_HandSolder, F.Cu at (180.0, 52.0)
- added C50: 10uF, Capacitor_SMD:C_0805_2012Metric_Pad1.18x1.45mm_HandSolder, F.Cu at (134.0, 62.0)
- added COMS1: Conn_01x05, Connector_PinHeader_2.54mm:PinHeader_1x05_P2.54mm_Vertical_SMD_Pin1Right, F.Cu at (151.0, 98.0)
- added D10: D_Schottky, Diode_SMD:D_SOD-323_HandSoldering, F.Cu at (141.0, 88.0)
- added J1: Conn_02x24_Odd_Even, Connector_PinHeader_2.54mm:PinHeader_2x24_P2.54mm_Vertical, F.Cu at (132.6, 58.6)
- added J3: USB_C_Receptacle_USB2.0_16P, USB4940-00-A:USB494000A, F.Cu at (144.0, 66.0)
- added MAIN1: Conn_01x05, Connector_PinHeader_2.54mm:PinHeader_1x05_P2.54mm_Vertical_SMD_Pin1Right, F.Cu at (165.0, 98.0)
- added R14: 26.1K, Resistor_SMD:R_0805_2012Metric_Pad1.20x1.40mm_HandSolder, F.Cu at (185.0, 49.0)
- added R16: 10k, Resistor_SMD:R_0805_2012Metric_Pad1.20x1.40mm_HandSolder, F.Cu at (145.0, 85.0)
- added R17: 10k, Resistor_SMD:R_0805_2012Metric_Pad1.20x1.40mm_HandSolder, F.Cu at (146.0, 82.0)
- added R18: 10k, Resistor_SMD:R_0805_2012Metric_Pad1.20x1.40mm_HandSolder, F.Cu at (174.0, 109.0)
- added R19: 10k, Resistor_SMD:R_0805_2012Metric_Pad1.20x1.40mm_HandSolder, F.Cu at (179.0, 108.0)
- added R6: 10k, Resistor_SMD:R_0805_2012Metric_Pad1.20x1.40mm_HandSolder, F.Cu at (186.0, 104.0)
- added R7: 120, Resistor_SMD:R_0805_2012Metric_Pad1.20x1.40mm_HandSolder, F.Cu at (191.0, 100.0)
- added RESET1: Conn_01x05, Connector_PinHeader_2.54mm:PinHeader_1x05_P2.54mm_Vertical_SMD_Pin1Right, F.Cu at (158.0, 98.0)
- added U7: AMS1117-3.3, Package_TO_SOT_SMD:SOT-223-3_TabPin2, F.Cu at (143.0, 76.0)
- C51: value 100nF -> 10uF
- C55: footprint XTAL_NX3215SA_NDK:XTAL_NX3215SA_NDK -> Capacitor_SMD:C_0805_2012Metric_Pad1.18x1.45mm_HandSolder
- C57: footprint TMUX1574PWR:PWP16_2P31X2P46_TEX -> Capacitor_SMD:C_0805_2012Metric_Pad1.18x1.45mm_HandSolder
- C60: footprint Capacitor_SMD:C_Elec_6.3x7.7 -> Capacitor_Tantalum_SMD:CP_EIA-7343-31_Kemet-D_HandSolder
- R20: value 10K -> 10k
- moved R10 172.7 mm to (204.0, 69.0)
- moved C29 172.6 mm to (199.0, 81.0)
- moved C19 170.5 mm to (204.0, 75.0)
- moved C12 167.7 mm to (199.0, 78.0)
- moved C22 167.0 mm to (194.0, 72.0)
- moved R8 166.1 mm to (204.0, 89.0)
- moved C4 165.1 mm to (199.0, 102.0)
- moved R9 165.0 mm to (204.0, 99.0)
- moved C10 164.2 mm to (199.0, 63.0)
- moved C24 164.1 mm to (199.0, 90.0)
- moved R3 163.5 mm to (204.0, 72.0)
- moved C27 163.2 mm to (199.0, 105.0)
- moved C11 163.1 mm to (194.0, 69.0)
- moved C3 163.1 mm to (199.0, 66.0)
- moved C9 163.1 mm to (199.0, 87.0)
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Connections:
- net +5V renamed 5V
- C51 pad 1: +3V3 -> Net-(D10-A)
Routing:
- net (no net): track 1.75 -> 0.00 mm
Other:
- board outline added: 93.5 x 94.8 mm

Commit message: I2C fixed
Parts:
- removed U12: TMUX1574PWR, TMUX1574PWR:PWP16_2P31X2P46_TEX
- added H1: MountingHole, MountingHole:MountingHole_3.2mm_M3_DIN965_Pad, F.Cu at (115.7, 50.0)
- added H2: MountingHole, MountingHole:MountingHole_3.2mm_M3_DIN965_Pad, F.Cu at (185.7, 50.0)
- added H3: MountingHole, MountingHole:MountingHole_3.2mm_M3_DIN965_Pad, F.Cu at (115.7, 120.0)
- added H4: MountingHole, MountingHole:MountingHole_3.2mm_M3_DIN965_Pad, F.Cu at (185.7, 120.0)
- added U8: TMUX1574PWR, TMUX1574PWR:SOP65P640X120-16N, F.Cu at (173.9, 66.1)
- J1: footprint Connector_PinHeader_2.54mm:PinHeader_2x24_P2.54mm_Vertical -> ESQ-124-38-L-D:ESQ-124-Y-X-D
- U10: footprint TMUX1574PWR:PWP16_2P31X2P46_TEX -> TMUX1574PWR:SOP65P640X120-16N
- moved C50 145.6 mm to (255.3, 142.5)
- moved R17 144.1 mm to (277.6, 140.8)
- moved R16 142.7 mm to (277.6, 137.8)
- moved C51 130.7 mm to (255.3, 145.5)
- moved D10 129.4 mm to (255.4, 148.5)
- moved SwReset3 128.6 mm to (249.9, 117.7)
- moved C55 126.2 mm to (272.8, 130.8)
- moved U7 124.1 mm to (247.9, 142.2)
- moved IC1 123.5 mm to (245.6, 148.6)
- moved C45 119.9 mm to (239.8, 107.6)
- moved SwReset2 115.5 mm to (212.6, 152.3)
- moved C30 115.4 mm to (202.4, 142.3)
- moved C48 115.4 mm to (255.3, 139.5)
- moved U6 112.3 mm to (240.2, 146.2)
- moved R18 109.3 mm to (277.6, 143.7)
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Connections:
- U10 pad 1: /Memory/select_py -> /Memory/select_coms
- U10 pad 12: /Memory/py_flash_clk_m -> /Memory/coms_flash_clk_m
- U10 pad 7: /Memory/py_flash_miso_m -> /Memory/coms_flash_miso_m
- U10 pad 9: /Memory/py_flash_mosi_m -> /Memory/coms_flash_mosi_m
Other:
- board size 93.5 x 94.8 mm -> 81 x 81 mm

Commit message: Finishing schematics
Parts:
- added C49: 100nF, Capacitor_SMD:C_0603_1608Metric_Pad1.08x0.95mm_HandSolder, F.Cu at (86.6, 152.6)
- added C52: 100nF, Capacitor_SMD:C_0603_1608Metric_Pad1.08x0.95mm_HandSolder, F.Cu at (81.9, 160.0)
- added R15: 4.7k, Resistor_SMD:R_0805_2012Metric_Pad1.20x1.40mm_HandSolder, F.Cu at (131.2, 139.3)
- added R21: 4.7k, Resistor_SMD:R_0805_2012Metric_Pad1.20x1.40mm_HandSolder, F.Cu at (131.2, 142.3)
- added R22: 10k, Resistor_SMD:R_0805_2012Metric_Pad1.20x1.40mm_HandSolder, F.Cu at (82.1, 146.1)
- added R23: 120, Resistor_SMD:R_0805_2012Metric_Pad1.20x1.40mm_HandSolder, F.Cu at (82.1, 149.1)
- added R24: 330, Resistor_SMD:R_0805_2012Metric_Pad1.20x1.40mm_HandSolder, F.Cu at (82.1, 157.3)
- added R25: 330, Resistor_SMD:R_0805_2012Metric_Pad1.20x1.40mm_HandSolder, F.Cu at (82.1, 152.0)
- added U12: SN65HVD230DR, SN65HVD230DR:D8, F.Cu at (99.2, 146.1)
- moved COMS1 47.1 mm to (159.9, 145.2)
- moved U1 1.85 mm to (151.9, 101.4)
Connections:
- net /Main/BOOT0 renamed /Main/BootMain
- net /Power MCU/BOOT0 renamed /Power MCU/BootRst
- C14 pad 1: SWD_NRST -> /Main/SWNRST
- C30 pad 1: SWD_NRST -> /Coms/SWNRST_Com
- COMS1 pad 2: /Power and Protections/SWCLK_Com -> /Coms/SWCLK_Com
- COMS1 pad 3: /Power and Protections/SWDIO_Com -> /Coms/SWDIO_Com
- COMS1 pad 4: /Power and Protections/SWNRST_Com -> /Coms/SWNRST_Com
- D3 pad 1: 5V -> +5V
- J1 pad 14: GND -> SW1
- J1 pad 15: SW1 -> EN_PY2
- J1 pad 17: EN_PY2 -> EN_COMS
- J1 pad 18: EN_COMS -> EN_QUEMADOR
- J1 pad 19: EN_ADCS -> EN_PY1
- J1 pad 2: +Vbatt -> NR
- J1 pad 20: EN_PY1 -> EN_ADCS
- J1 pad 21: GND -> EN_ADCS_5V
- J1 pad 22: EN_ADCS_5V -> GND
- J1 pad 23: Can_H -> GND
- J1 pad 24: GND -> CAN_H
- J1 pad 25: Can_L -> GND
- J1 pad 26: GND -> CAN_L
- J1 pad 27: I2C_SDA -> I2C_SCL
- J1 pad 28: I2C_SCL -> I2C_SDA
- J1 pad 31: GND -> Interrupción EPS
- J1 pad 32: Interrupción EPS -> GND
- J1 pad 33: EN_OBC -> GND
- J1 pad 34: GND -> EN_OBC
- J1 pad 37: PY2_RX -> PY2_TX
- J1 pad 38: PY2_TX -> PY2_RX
- J1 pad 40: GND -> CS_PY2
- J1 pad 41: SPI_MOSI -> CS_COMS
- J1 pad 42: unconnected-(J1-Pin_42-Pad42) -> SPI_MOSI
- J1 pad 43: SPI_SCK -> SPI_MISO
- J1 pad 44: unconnected-(J1-Pin_44-Pad44) -> SPI_SCK
- J1 pad 47: COMS_RX -> ObcComs_TX
- J1 pad 48: COMS_TX -> ComsOBC_RX
- MAIN1 pad 2: /Power and Protections/SWCLK -> /Main/SWCLK
- MAIN1 pad 3: /Power and Protections/SWDIO -> /Main/SWDIO
- MAIN1 pad 4: /Power and Protections/SWNRST -> /Main/SWNRST
- R10 pad 1: /Coms/LGreen -> /Coms/LGreenC
- R12 pad 1: /Power MCU/LRed -> /Power MCU/LRedP
- R13 pad 1: /Power MCU/LGreen -> /Power MCU/LGreenP
- R9 pad 1: /Coms/LRed -> /Coms/LRedC
- RESET1 pad 2: /Power and Protections/SWCLK_RST -> /Power MCU/SWCLK_RST
- RESET1 pad 3: /Power and Protections/SWDIO_RST -> /Power MCU/SWDIO_RST
- RESET1 pad 4: /Power and Protections/SWNRST_RST -> SWD_NRST
- SwReset1 pad 2: SWD_NRST -> /Main/SWNRST
- SwReset2 pad 2: SWD_NRST -> /Coms/SWNRST_Com
- U1 pad 14: Rst_TX -> MainPwr_TX
- U1 pad 15: Rst_RX -> MainPwr_RX
- U1 pad 37: unconnected-(U1-PC6-Pad37) -> SW2
- U1 pad 38: unconnected-(U1-PC7-Pad38) -> SW1
- U1 pad 40: unconnected-(U1-PC9-Pad40) -> EN_QUEMADOR
- U1 pad 42: Coms_TX -> MainComs_TX
- U1 pad 43: Coms_RX -> MainComs_RX
- U1 pad 46: SWDIO1 -> /Main/SWDIO
- U1 pad 49: SWCLK1 -> /Main/SWCLK
- U1 pad 50: unconnected-(U1-PA15-Pad50) -> CsMemPY
- U1 pad 51: unconnected-(U1-PC10-Pad51) -> EnMuxPy
- U1 pad 52: unconnected-(U1-PC11-Pad52) -> CsMemPY
- U1 pad 53: unconnected-(U1-PC12-Pad53) -> PY2_TX
- U1 pad 54: unconnected-(U1-PD2-Pad54) -> PY2_RX
- U1 pad 55: unconnected-(U1-PB3-Pad55) -> PY2_SCK
- U1 pad 56: unconnected-(U1-PB4-Pad56) -> PY2_MISO
- U1 pad 57: unconnected-(U1-PB5-Pad57) -> PY2_MOSI
- U1 pad 58: unconnected-(U1-PB6-Pad58) -> I2C_SCL
- U1 pad 59: unconnected-(U1-PB7-Pad59) -> I2C_SDA
- U1 pad 61: unconnected-(U1-PB8-Pad61) -> /Main/Can_RX
- U1 pad 62: unconnected-(U1-PB9-Pad62) -> /Main/Can_TX
- U1 pad 7: SWD_NRST -> /Main/SWNRST
- U1 pad 9: unconnected-(U1-PC1-Pad9) -> Interrupción EPS
- U10 pad 1: /Memory/select_coms -> EnMuxCom
- U10 pad 10: unconnected-(U10-S3B-Pad10) -> SPI_SCK
- U10 pad 11: unconnected-(U10-S3A-Pad11) -> ComMem_SCK
- U10 pad 12: /Memory/coms_flash_clk_m -> /Memory/cs_mem_py
- U10 pad 13: unconnected-(U10-S4B-Pad13) -> CS_COMS
- U10 pad 14: unconnected-(U10-S4A-Pad14) -> CsMemComs
- U10 pad 2: unconnected-(U10-S1A-Pad2) -> ComMem_MISO
- U10 pad 3: unconnected-(U10-S1B-Pad3) -> SPI_MISO
- U10 pad 4: unconnected-(U10-D1-Pad4) -> /Memory/coms_flash_miso_m
- U10 pad 5: unconnected-(U10-S2A-Pad5) -> ComMem_MOSI
- U10 pad 6: unconnected-(U10-S2B-Pad6) -> SPI_MOSI
- U10 pad 7: /Memory/coms_flash_miso_m -> /Memory/coms_flash_mosi_m
- U10 pad 9: /Memory/coms_flash_mosi_m -> /Memory/coms_flash_clk_m
- U11 pad 1: GND -> /Memory/cs_mem_py
- U3 pad 5: 5V -> +5V
- U4 pad 14: unconnected-(U4-PA0-Pad14) -> MainComs_RX
- U4 pad 15: unconnected-(U4-PA1-Pad15) -> MainComs_TX
- U4 pad 27: unconnected-(U4-PB1-Pad27) -> /Coms/LGreenC
- U4 pad 28: unconnected-(U4-PB2-Pad28) -> /Coms/LRedC
- U4 pad 42: Coms_RX -> unconnected-(U4-PA9-Pad42)
- U4 pad 43: Coms_TX -> unconnected-(U4-PA10-Pad43)
- U4 pad 44: unconnected-(U4-PA11-Pad44) -> /Coms/Can_RX
- U4 pad 45: unconnected-(U4-PA12-Pad45) -> /Coms/Can_TX
- U4 pad 46: SWDIO2 -> /Coms/SWDIO_Com
- U4 pad 49: SWCLK2 -> /Coms/SWCLK_Com
- U4 pad 51: unconnected-(U4-PC10-Pad51) -> ObcComs_TX
- U4 pad 52: unconnected-(U4-PC11-Pad52) -> ComsOBC_RX
- U4 pad 53: unconnected-(U4-PC12-Pad53) -> EnMuxCom
- U4 pad 54: unconnected-(U4-PD2-Pad54) -> CsMemComs
- U4 pad 55: unconnected-(U4-PB3-Pad55) -> ComMem_SCK
- U4 pad 56: unconnected-(U4-PB4-Pad56) -> ComMem_MISO
- U4 pad 57: unconnected-(U4-PB5-Pad57) -> ComMem_MOSI
- U4 pad 7: SWD_NRST -> /Coms/SWNRST_Com
- U5 pad 14: Rst_RX -> /Power MCU/LGreenP
- U5 pad 15: Rst_TX -> /Power MCU/LRedP
- U5 pad 22: unconnected-(U5-PA6-Pad22) -> watchdog
- U5 pad 23: set_0 -> unconnected-(U5-PA7-Pad23)
- U5 pad 24: set_1 -> unconnected-(U5-PC4-Pad24)
- U5 pad 25: set_2 -> unconnected-(U5-PC5-Pad25)
- U5 pad 33: unconnected-(U5-PB12-Pad33) -> MainRst
- U5 pad 35: unconnected-(U5-PB14-Pad35) -> ComsRst
- U5 pad 37: Rst_RX -> MainPwr_RX
- U5 pad 38: Rst_TX -> MainPwr_TX
- U5 pad 46: SWDIO3 -> /Power MCU/SWDIO_RST
- U5 pad 49: SWCLK3 -> /Power MCU/SWCLK_RST
- U5 pad 50: unconnected-(U5-PA15-Pad50) -> EN_ADCS_5V
- U6 pad 1: rst_wdi -> watchdog
- U6 pad 4: set_0 -> +3V3
- U6 pad 5: set_1 -> GND
- U6 pad 6: set_2 -> +3V3
- U7 pad 3: 5V -> +5V
- U8 pad 1: /Memory/select_py -> EnMuxPy
- U8 pad 10: unconnected-(U8-S3B-Pad10) -> SPI_SCK
- U8 pad 11: unconnected-(U8-S3A-Pad11) -> PY2_SCK
- U8 pad 12: /Memory/py_flash_mosi_m -> /Memory/cs_mem_py
- U8 pad 13: unconnected-(U8-S4B-Pad13) -> CS_PY2
- U8 pad 14: unconnected-(U8-S4A-Pad14) -> CsMemPY
- U8 pad 2: unconnected-(U8-S1A-Pad2) -> PY2_MISO
- U8 pad 3: unconnected-(U8-S1B-Pad3) -> SPI_MISO
- U8 pad 4: unconnected-(U8-D1-Pad4) -> /Memory/py_flash_miso_m
- U8 pad 5: unconnected-(U8-S2A-Pad5) -> PY2_MOSI
- U8 pad 6: unconnected-(U8-S2B-Pad6) -> SPI_MOSI
- U8 pad 7: /Memory/py_flash_miso_m -> /Memory/py_flash_mosi_m
- U9 pad 1: GND -> /Memory/cs_mem_py

Commit message: Placement
Parts:
- removed R23: 120, Resistor_SMD:R_0805_2012Metric_Pad1.20x1.40mm_HandSolder
- moved C49 162.9 mm to (222.4, 62.6), turned to 180 degrees
- moved R22 162.0 mm to (217.8, 57.6), turned to 90 degrees
- moved C50 159.3 mm to (117.5, 62.6), turned to -90 degrees
- moved U12 151.5 mm to (222.1, 57.5), turned to 90 degrees
- moved IC1 150.9 mm to (121.8, 62.5)
- moved R16 148.5 mm to (146.0, 69.0), turned to -90 degrees
- moved SwBoot3 144.8 mm to (113.6, 91.0), turned to 180 degrees
- moved R20 144.0 mm to (121.8, 59.5)
- moved D6 143.2 mm to (113.8, 107.2)
- moved D7 143.2 mm to (113.8, 110.3)
- moved R17 138.8 mm to (158.2, 69.9), turned to -90 degrees
- moved R14 138.5 mm to (121.8, 65.8), turned to 180 degrees
- moved SwReset3 136.5 mm to (114.5, 101.0)
- moved C60 135.5 mm to (127.2, 62.8), turned to -90 degrees
- moved XTAL3 132.8 mm to (122.6, 80.6)
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Routing:
- net /Main/LSE_OUT: track 0.00 -> 11.2 mm
- net /Main/LSE_IN: track 0.00 -> 8.87 mm
- net /Main/HSE_IN: track 0.00 -> 8.67 mm
- net /Main/HSE_OUT: track 0.00 -> 6.37 mm
- net +3V3A: track 0.00 -> 5.11 mm
- net GND: track 0.00 -> 2.13 mm
- net +3V3: track 0.00 -> 2.08 mm
- added copper zone on In1.Cu, net GND
Other:
- copper layers 2 -> 4

Commit message: PC104
Parts:
- moved C48 0.33 mm to (127.7, 103.1)
- moved U6 0.33 mm to (129.5, 99.4)
Changed lines of the file:
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@@
 	)
 	(footprint "ESQ-124-38-L-D:ESQ-124-Y-X-D"
+		(locked yes)
 		(layer "F.Cu")
 		(at 121.506655 48.713416 180)
@@
 			)
 		)
-		(fp_text user "*"
-			(at -1.6129 -2.4257 90)
+		(fp_text user "${REFERENCE}"
+			(at 0 0 90)
+			(unlocked yes)
 			(layer "F.Fab")
 			(effects
@@
 			)
 		)
-		(fp_text user "${REFERENCE}"
-			(at 0 0 90)
-			(unlocked yes)
+		(fp_text user "*"
+			(at -1.6129 -2.4257 90)
 			(layer "F.Fab")
 			(effects
@@
 		)
 		(embedded_fonts no)
+		(model "${KIPRJMOD}/assets/ul_SN65HVD230DR/D0008A.stp"
+			(offset
+				(xyz 0 0 0)
+			)
+			(scale
+				(xyz 1 1 1)
+			)
+			(rotate
+				(xyz 0 0 0)
+			)
+		)
 	)
 	(footprint "Capacitor_SMD:C_0805_2012Metric_Pad1.18x1.45mm_HandSolder"
@@
 	(footprint "Capacitor_SMD:C_0805_2012Metric_Pad1.18x1.45mm_HandSolder"
 		(layer "F.Cu")
-		(at 128.037501 103.113149 180)
+		(at 127.7125 103.113149 180)
 		(descr "Capacitor SMD 0805 (2012 Metric), square (rectangular) end terminal, IPC-7351 nominal with elongated pad for handsoldering. (Body size source: IPC-SM-782 page 76, https://www.pcb-3d.com/wordpress/wp-content/uploads/ipc-sm-782a_amendment_1_and_2.pdf, https://docs.google.com/spreadsheets/d/1BsfQQcO9C6DZCsRaXUlFlo91Tg2WpOkGARC1WS5S8t0/edit?usp=sharing), generated with kicad-footprint-generator")
 		(tags "capacitor handsolder")
@@
 		)
 		(fp_circle
-			(center -2.2 1.3)
-			(end -2.1238 1.3)
+			(center -2.8067 0)
+			(end -2.7305 0)
 			(stroke
 				(width 0.1524)
@@
 	(footprint "MAX6369KA+T:21-0078H_MXM"
 		(layer "F.Cu")
-		(at 129.825001 99.363149 -90)
+		(at 129.5 99.363149 -90)
 		(tags "MAX6369KA+T ")
 		(property "Reference" "U6"
@@
 		)
 		(fp_text user "*"
-			(at -1.617149 -2.549 90)
+			(at -1.617149 -2.549 270)
+			(unlocked yes)
 			(layer "F.SilkS")
 			(effects
@@
 		)
 		(fp_text user "*"
-			(at -0.4953 -1.4224 90)
+			(at -0.4953 -1.4224 270)
+			(unlocked yes)
 			(layer "F.Fab")
 			(effects
@@
 		)
 		(embedded_fonts no)
+		(model "${KIPRJMOD}/assets/TMUX1574PWR/TMUX1574PWR.step"
+			(offset
+				(xyz 0 0 0)
+			)
+			(scale
+				(xyz 1 1 1)
+			)
+			(rotate
+				(xyz -90 -0 -0)
+			)
+		)
 	)
 	(footprint "Resistor_SMD:R_0805_2012Metric_Pad1.20x1.40mm_HandSolder"
@@
 		)
 		(fp_text user "*"
-			(at -4.2141 -2.6356 90)
+			(at -3.8989 -3.5806 90)
 			(layer "F.SilkS")
 			(effects
@@
 		(fp_text user "*"
 			(at -2.286 -2.5908 90)
+			(unlocked yes)
 			(layer "F.Fab")
 			(effects
@@
 		)
 		(embedded_fonts no)
-		(model "${KIPRJMOD}/Footprints/ul_W25Q128JVSIQ/SOIC_128JVSIQ_WIN.step"
+		(model "${KIPRJMOD}/assets/ul_W25Q128JVSIQ/SOIC_128JVSIQ_WIN.step"
 			(offset
 				(xyz 0 0 0)
@@
 		)
 		(embedded_fonts no)
+		(model "${KIPRJMOD}/assets/TMUX1574PWR/TMUX1574PWR.step"
+			(offset
+				(xyz 0 0 0)
+			)
+			(scale
+				(xyz 1 1 1)
+			)
+			(rotate
+				(xyz -90 -0 -0)
+			)
+		)
 	)
 	(footprint "OCP_TPS2553QDBVRQ1:SOT95P280X145-6N"
@@
 		(fp_text user "*"
 			(at -2.286 -2.5908 0)
-			(unlocked yes)
 			(layer "F.Fab")
 			(effects
@@
 			)
 		)
-		(fp_text user "*"
-			(at -2.286 -2.5908 0)
+		(fp_text user "${REFERENCE}"
+			(at 0 0 0)
+			(unlocked yes)
 			(layer "F.Fab")
 			(effects
@@
 			)
 		)
-		(fp_text user "${REFERENCE}"
-			(at 0 0 0)
+		(fp_text user "*"
+			(at -2.286 -2.5908 0)
 			(unlocked yes)
 			(layer "F.Fab")
@@
 		)
 		(embedded_fonts no)
-		(model "${KIPRJMOD}/Footprints/ul_W25Q128JVSIQ/SOIC_128JVSIQ_WIN.step"
+		(model "${KIPRJMOD}/assets/ul_W25Q128JVSIQ/SOIC_128JVSIQ_WIN.step"
 			(offset
 				(xyz 0 0 0)
@@
 		(fp_text user "*"
 			(at -2.97535 -3.606 90)
-			(unlocked yes)
 			(layer "F.SilkS")
 			(effects
@@
 		)
 		(embedded_fonts no)
+		(model "${KIPRJMOD}/assets/ul_SN65HVD230DR/D0008A.stp"
+			(offset
+				(xyz 0 0 0)
+			)
+			(scale
+				(xyz 1 1 1)
+			)
+			(rotate
+				(xyz 0 0 0)
+			)
+		)
 	)
 	(gr_line
