File: PCB/OBC/OBC.kicad_pcb (KiCad board)
At the start: 4 copper layers, 81 x 81 mm, 126 parts, among them IC1 TPS2553QDBVRQ1, J1 Conn_02x24_Odd_Even, J3 USB_C_Receptacle_USB2.0_16P, U1 STM32F405RGTx, U10 TMUX1574PWR, U11 W25Q128JVSIQ, U12 SN65HVD230DR, U2 SN65HVD230DR, U3 USBLC6-2SC6, U4 STM32F405RGTx, U5 STM32F405RGTx, U6 MAX6369KA+T, U7 AMS1117-3.3, U8 TMUX1574PWR, U9 W25Q128JVSIQ

Commit message: Add some netclasses
Parts:
- added D8: D_Schottky, Diode_SMD:D_SOD-323_HandSoldering, F.Cu at (119.0, 75.7)
- added D9: D_Schottky, Diode_SMD:D_SOD-323_HandSoldering, F.Cu at (149.5, 116.0)
- C11, C22, C26, C37, C41, C6: footprint Capacitor_SMD:C_0805_2012Metric_Pad1.18x1.45mm_HandSolder -> Capacitor_SMD:C_0603_1608Metric_Pad1.08x0.95mm_HandSolder
- moved C16 9.69 mm to (142.7, 107.9)
- moved FB1 7.79 mm to (134.0, 107.9)
- moved C60 2.82 mm to (125.0, 64.5)
- moved IC1 2.82 mm to (119.5, 64.3)
- moved R14 2.82 mm to (119.5, 67.5)
- moved C50 2.82 mm to (115.3, 64.3)
- moved R20 2.82 mm to (119.5, 61.3)
- moved C47 1.78 mm to (121.7, 87.6), turned to -90 degrees
- moved C26 1.58 mm to (175.6, 89.0)
- moved C42 1.35 mm to (134.8, 91.5), turned to -90 degrees
- moved C8 1.26 mm to (140.7, 107.9)
- moved C5 1.24 mm to (138.5, 107.9)
- moved C24 1.23 mm to (176.2, 76.3)
- moved C17 1.22 mm to (136.2, 107.9)
- moved C41 1.21 mm to (138.3, 89.7)
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Connections:
- COMS1 pad 1: +3V3 -> d3v3
- J1 pad 27: I2C_SCL -> GND
- J1 pad 28: I2C_SDA -> GND
- J1 pad 29: GND -> I2C_SCL
- J1 pad 30: GND -> I2C_SDA
- MAIN1 pad 1: +3V3 -> d3v3
- RESET1 pad 1: +3V3 -> Net-(D8-A)
Routing:
- net +3V3: track 2.08 -> 45.3 mm
- net GND: track 2.13 -> 35.2 mm
- net MainPwr_RX: track 0.00 -> 28.6 mm, vias 0 -> 2
- net MainPwr_TX: track 0.00 -> 27.4 mm, vias 0 -> 2
- net MainComs_TX: track 0.00 -> 22.5 mm, vias 0 -> 2
- net MainComs_RX: track 0.00 -> 22.2 mm, vias 0 -> 2
- net +3V3A: track 5.11 -> 26.4 mm
- net /Coms/SWCLK_Com: track 0.00 -> 15.4 mm
- net /Coms/SWDIO_Com: track 0.00 -> 13.2 mm
- net /Coms/HSE_IN: track 0.00 -> 9.30 mm
- net /Power MCU/HSE_IN: track 0.00 -> 8.27 mm
- net /Coms/HSE_OUT: track 0.00 -> 6.65 mm
- net /Power MCU/HSE_OUT: track 0.00 -> 5.60 mm
- net Net-(U1-VCAP_2): track 0.00 -> 3.03 mm
- net Net-(U5-VCAP_2): track 0.00 -> 2.99 mm
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
Commit message: Coms memory finished
Parts:
- removed J1: Conn_02x24_Odd_Even, ESQ-124-38-L-D:ESQ-124-Y-X-D
- removed R7: 120, Resistor_SMD:R_0805_2012Metric_Pad1.20x1.40mm_HandSolder
- added C59: 4.7 nF, Capacitor_SMD:C_0805_2012Metric_Pad1.18x1.45mm_HandSolder, F.Cu at (150.4, 56.1)
- added J2: Conn_02x24_Odd_Even, KiCad:ESQ-124-Y-X-D, F.Cu at (121.2, 48.3)
- added R23: 60, Resistor_SMD:R_0603_1608Metric_Pad0.98x0.95mm_HandSolder, F.Cu at (149.5, 59.2)
- added R26: 60, Resistor_SMD:R_0603_1608Metric_Pad0.98x0.95mm_HandSolder, F.Cu at (151.3, 60.8)
- C49, C53, C54, C55, R16, R17, R22, U12, U8, U9: moved to B.Cu
- moved U12 64.1 mm to (158.6, 66.4), turned to -90 degrees
- moved C49 63.8 mm to (158.6, 61.4)
- moved R22 60.8 mm to (158.6, 71.6), turned to 180 degrees
- moved U8 25.0 mm to (153.4, 86.0), turned to 90 degrees
- moved C53 21.7 mm to (155.5, 80.7), turned to 180 degrees
- moved R17 20.7 mm to (142.8, 83.7), turned to 90 degrees
- moved R16 19.5 mm to (142.8, 88.3), turned to 90 degrees
- moved U9 19.4 mm to (147.0, 86.2), turned to 90 degrees
- moved C55 18.8 mm to (148.1, 79.8), turned to 180 degrees
- moved R6 16.8 mm to (146.3, 66.3)
- moved U2 16.8 mm to (150.3, 66.3)
- moved C54 15.6 mm to (148.1, 77.5), turned to 180 degrees
- moved C52 12.3 mm to (150.3, 71.5), turned to 180 degrees
- moved D10 9.22 mm to (165.5, 101.9), turned to 90 degrees
- moved C50 8.57 mm to (121.1, 58.0), turned to 180 degrees
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Connections:
- U10 pad 12: /Memory/cs_mem_py -> /Memory/cs_mem_coms
- U11 pad 1: /Memory/cs_mem_py -> /Memory/cs_mem_coms
- U2 pad 5: unconnected-(U2-VREF-Pad5) -> Net-(U2-VREF)
Routing:
- net +3V3: track 45.3 -> 130.6 mm
- net GND: track 35.2 -> 105.4 mm, vias 0 -> 39
- net EN_OBC: track 0.00 -> 59.8 mm
- net /Coms/SWNRST_Com: track 0.00 -> 46.4 mm, vias 0 -> 2
- net ObcComs_TX: track 0.00 -> 43.8 mm
- net ComsOBC_RX: track 0.00 -> 40.3 mm
- net EN_PY1: track 0.00 -> 33.4 mm
- net EN_ADCS_5V: track 0.00 -> 33.0 mm, vias 0 -> 1
- net EN_COMS: track 0.00 -> 32.1 mm
- net SWD_NRST: track 0.00 -> 31.9 mm, vias 0 -> 2
- net EN_PY2: track 0.00 -> 31.5 mm
- net /Power MCU/LGreenP: track 0.00 -> 30.5 mm, vias 0 -> 2
- net EN_ADCS: track 0.00 -> 30.2 mm
- net /Power MCU/SWCLK_RST: track 0.00 -> 29.7 mm
- net /Power MCU/SWDIO_RST: track 0.00 -> 26.7 mm, vias 0 -> 2
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- added copper zone on In2.Cu, net GND
