File: PCB/OBC/storage.kicad_sch (KiCad schematic)
At the start: 10 parts, among them IC1 TPS2553QDBVRQ1, U6 MAX6369KA+T, U7 AMS1117-3.3

Commit message: Coms memory finished
Changed lines of the file:
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@@
 	(wire
 		(pts
-			(xy 176.53 46.99) (xy 176.53 48.26)
+			(xy 161.29 46.99) (xy 161.29 48.26)
 		)
 		(stroke
@@
 	(wire
 		(pts
-			(xy 176.53 48.26) (xy 180.34 48.26)
+			(xy 161.29 48.26) (xy 180.34 48.26)
 		)
 		(stroke
@@
 	(symbol
 		(lib_id "power:+5V")
-		(at 176.53 46.99 0)
+		(at 161.29 46.99 0)
 		(unit 1)
 		(exclude_from_sim no)
@@
 		(fields_autoplaced yes)
 		(property "Reference" "#PWR077"
-			(at 176.53 50.8 0)
+			(at 161.29 50.8 0)
 			(effects
 				(font
@@
 		)
 		(property "Value" "+5V"
-			(at 176.53 41.91 0)
+			(at 161.29 41.91 0)
 			(effects
 				(font
@@
 		)
 		(property "Footprint" ""
-			(at 176.53 46.99 0)
+			(at 161.29 46.99 0)
 			(effects
 				(font
@@
 		)
 		(property "Datasheet" ""
-			(at 176.53 46.99 0)
+			(at 161.29 46.99 0)
 			(effects
 				(font
@@
 		)
 		(property "Description" "Power symbol creates a global label with name \"+5V\""
-			(at 176.53 46.99 0)
-			(effects
-				(font
+			(at 161.29 46.99 0)
+			(effects
+				(font

Commit message: Routing finished, without errors
Parts:
- added C61: 10uF, Capacitor_SMD:C_0805_2012Metric_Pad1.18x1.45mm_HandSolder, symbol Device:C
Connections:
- net GND: now also C61.2
- net at C51.1, D10.2 (A), U7.2 (VO): now also C61.1
Other:
- moved on the sheet: D10
Changed lines of the file:
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@@
+	)
+	(junction
+		(at 199.39 55.88)
+		(diameter 0)
+		(color 0 0 0 0)
+	)
+	(junction
+		(at 204.47 48.26)
+		(diameter 0)
+		(color 0 0 0 0)
 	)
 	(junction
@@
 	(wire
 		(pts
-			(xy 213.36 48.26) (xy 207.01 48.26)
+			(xy 213.36 48.26) (xy 212.09 48.26)
 		)
 		(stroke
@@
 	(wire
 		(pts
+			(xy 199.39 55.88) (xy 204.47 55.88)
+		)
+		(stroke
+			(width 0)
+			(type default)
+		)
+	)
+	(wire
+		(pts
 			(xy 45.72 93.98) (xy 45.72 99.06)
+		)
+		(stroke
+			(width 0)
+			(type default)
+		)
+	)
+	(wire
+		(pts
+			(xy 204.47 48.26) (xy 199.39 48.26)
 		)
 		(stroke
@@
 		(dnp no)
 		(property "Reference" "C51"
-			(at 202.184 51.054 0)
+			(at 201.168 59.436 0)
 			(effects
 				(font
@@
 		)
 		(property "Value" "10uF"
-			(at 202.184 53.594 0)
+			(at 201.168 61.976 0)
 			(effects
 				(font
@@
 	(symbol
 		(lib_id "Device:D_Schottky")
-		(at 203.2 48.26 180)
+		(at 208.28 48.26 180)
 		(unit 1)
 		(exclude_from_sim no)
@@
 		(dnp no)
 		(property "Reference" "D10"
-			(at 205.232 35.56 90)
+			(at 210.312 35.56 90)
 			(effects
 				(font
@@
 		)
 		(property "Value" "D_Schottky"
-			(at 202.692 35.56 90)
+			(at 207.772 35.56 90)
 			(effects
 				(font
@@
 		)
 		(property "Footprint" "Diode_SMD:D_SOD-323_HandSoldering"
-			(at 203.2 48.26 0)
+			(at 208.28 48.26 0)
 			(effects
 				(font
@@
 		)
 		(property "Datasheet" "~"
-			(at 203.2 48.26 0)
+			(at 208.28 48.26 0)
 			(effects
 				(font
@@
 		)
 		(property "Description" "Schottky diode"
-			(at 203.2 48.26 0)
+			(at 208.28 48.26 0)
 			(effects
 				(font
@@
 		)
 		(property "Availability" ""
-			(at 203.2 48.26 90)
+			(at 208.28 48.26 90)
 			(effects
 				(font
@@
 		)
 		(property "Check_prices" ""
-			(at 203.2 48.26 90)
+			(at 208.28 48.26 90)
 			(effects
 				(font
@@
 		)
 		(property "Description_1" ""
-			(at 203.2 48.26 90)
+			(at 208.28 48.26 90)
 			(effects
 				(font
@@
 		)
 		(property "MF" ""
-			(at 203.2 48.26 90)
+			(at 208.28 48.26 90)
 			(effects
 				(font
@@
 		)
 		(property "MP" ""
-			(at 203.2 48.26 90)
+			(at 208.28 48.26 90)
 			(effects
 				(font
@@
 		)
 		(property "Package" ""
-			(at 203.2 48.26 90)
+			(at 208.28 48.26 90)
 			(effects
 				(font
@@
 		)
 		(property "Price" ""
-			(at 203.2 48.26 90)
+			(at 208.28 48.26 90)
 			(effects
 				(font
@@
 		)
 		(property "SnapEDA_Link" ""
-			(at 203.2 48.26 90)
+			(at 208.28 48.26 90)
 			(effects
 				(font
@@
 		)
 		(property "Mouser" ""
-			(at 203.2 48.26 90)
+			(at 208.28 48.26 90)
 			(effects
 				(font
@@
 		)
 		(property "LCSC Part Name" "C124187"
-			(at 203.2 48.26 90)
+			(at 208.28 48.26 90)
 			(effects
 				(font
@@
 					(unit 1)
 				)
+			)
+		)
+	)
+	(symbol
+		(lib_id "Device:C")
+		(at 204.47 52.07 0)
+		(unit 1)
+		(exclude_from_sim no)
+		(in_bom yes)
+		(on_board yes)
+		(dnp no)
+		(property "Reference" "C61"
+			(at 206.248 59.436 0)
+			(effects
+				(font
+					(size 1.27 1.27)
+				)
+				(justify left)
+			)
+		)
+		(property "Value" "10uF"
+			(at 206.248 61.976 0)
+			(effects
+				(font
+					(size 1.27 1.27)
+				)
+				(justify left)
+			)
+		)
+		(property "Footprint" "Capacitor_SMD:C_0805_2012Metric_Pad1.18x1.45mm_HandSolder"
+			(at 205.4352 55.88 0)
+			(effects
+				(font
+					(size 1.27 1.27)
+				)
+				(hide yes)
+			)
+		)
+		(property "Datasheet" "~"
+			(at 204.47 52.07 0)
+			(effects
+				(font
+					(size 1.27 1.27)
+				)
+				(hide yes)
+			)
+		)
+		(property "Description" "Unpolarized capacitor"
+			(at 204.47 52.07 0)
+			(effects
+				(font
+					(size 1.27 1.27)
+				)
+				(hide yes)
+			)
+		)
+		(property "KLC_S3.3" ""
+			(at 204.47 52.07 0)
+			(effects
+				(font
+					(size 1.27 1.27)
+				)
+				(hide yes)
+			)
+		)
+		(property "KLC_S4.1" ""
+			(at 204.47 52.07 0)
+			(effects
+				(font
+					(size 1.27 1.27)
+				)
+				(hide yes)
+			)
+		)
+		(property "Sim.Device" ""
+			(at 204.47 52.07 0)
+			(effects
+				(font
+					(size 1.27 1.27)
+				)
+				(hide yes)
+			)
+		)
+		(property "Sim.Type" ""
+			(at 204.47 52.07 0)
+			(effects
+				(font
+					(size 1.27 1.27)
+				)
+				(hide yes)
+			)
+		)
+		(property "LCSC Part Name" "C237493"
+			(at 204.47 52.07 0)
+			(effects
+				(font
+					(size 1.27 1.27)
+				)
+				(hide yes)
+			)
+		)
+		(pin "1"
+		)
+		(pin "2"
+		)
+		(instances
+			(project "OBC"
+				(path "/e2c03eef-3b12-44a7-ba52-633d5337a24a/50cd9bda-d2af-42b5-bb85-974edeb725b5"
+					(reference "C61")
+					(unit 1)
+				)
