File: PCB/PCB_Interno/PCB_Interno.kicad_sch (KiCad schematic)
At the start: 5 parts, among them J1 Conn_02x24_Odd_Even

Commit message: I2C fixed
Parts:
- removed J1: Conn_02x24_Odd_Even, ESQ-124-38-L-D:ESQ-124-Y-X-D, symbol Connector_Generic:Conn_02x24_Odd_Even
- added J2: Conn_02x24_Odd_Even, KiCad:ESQ-124-Y-X-D, symbol Connector_Generic:Conn_02x24_Odd_Even
Connections:
- net +Vbatt: now also J2.1 (Pin_1), J2.2 (Pin_2), J2.5 (Pin_5), J2.6 (Pin_6)
- net 5V: now also J2.10 (Pin_10), J2.9 (Pin_9)
- net Can_H: now also J2.24 (Pin_24)
- net Can_L: now also J2.26 (Pin_26)
- net EN_ADCS: now also J2.20 (Pin_20)
- net EN_ADCS_5V: now also J2.21 (Pin_21)
- net EN_COMS: now also J2.17 (Pin_17)
- net EN_OBC: now also J2.34 (Pin_34)
- net EN_PY1: now also J2.19 (Pin_19)
- net EN_PY2: now also J2.18 (Pin_18)
- net GND: now also J2.11 (Pin_11), J2.12 (Pin_12), J2.13 (Pin_13), J2.14 (Pin_14), J2.22 (Pin_22), J2.23 (Pin_23), J2.25 (Pin_25), J2.29 (Pin_29), J2.3 (Pin_3), J2.30 (Pin_30), J2.32 (Pin_32), J2.33 (Pin_33), J2.35 (Pin_35), J2.36 (Pin_36), J2.39 (Pin_39), J2.4 (Pin_4), J2.40 (Pin_40), J2.45 (Pin_45), J2.46 (Pin_46), J2.7 (Pin_7), J2.8 (Pin_8)
- net I2C_SCL: now also J2.27 (Pin_27)
- net I2C_SDA: now also J2.28 (Pin_28)
- net Interrupción EPS: now also J2.31 (Pin_31)
- net PY2_RX: now also J2.38 (Pin_38)
- net PY2_TX: now also J2.37 (Pin_37)
- net SPI_MOSI: now also J2.42 (Pin_42)
- net SPI_SCK: now also J2.44 (Pin_44)
- net SW1: now also J2.16 (Pin_16)
- net SW2: now also J2.15 (Pin_15)
- new net COMS_RX: J2.48 (Pin_48)
- new net COMS_TX: J2.47 (Pin_47)
Other:
- removed sheet Coms
- removed sheet Main
- removed sheet Memory
- removed sheet Power MCU
- removed sheet Power and Protections
- moved on the sheet: H1, H2, H3, H4

Commit message: PC104
Connections:
- net +Vbatt: no longer J2.2 (Pin_2)
- net EN_PY2: now also J2.15 (Pin_15); no longer J2.18 (Pin_18)
- net GND: now also J2.27 (Pin_27), J2.28 (Pin_28); no longer J2.14 (Pin_14), J2.29 (Pin_29), J2.30 (Pin_30), J2.40 (Pin_40)
- net I2C_SCL: now also J2.29 (Pin_29); no longer J2.27 (Pin_27)
- net I2C_SDA: now also J2.30 (Pin_30); no longer J2.28 (Pin_28)
- net SPI_MISO: now also J2.43 (Pin_43)
- net SW1: now also J2.14 (Pin_14); no longer J2.16 (Pin_16)
- net SW2: now also J2.16 (Pin_16); no longer J2.15 (Pin_15)
- net CS_COMS: now reaches J2.41 (Pin_41)
- net COMS_RX renamed ComsOBC_RX
- net COMS_TX renamed ObcComs_TX
- net Can_H renamed CAN_H
- net Can_L renamed CAN_L
- new net CS_PY2: J2.40 (Pin_40)
- new net EN_QUEMADOR: J2.18 (Pin_18)
- new net NR: J2.2 (Pin_2)
